Commit message: Added support for Flir PTU-5.

File: clearpath_generator_common_tests/samples/test_all_dual_sensors/robot.urdf.xacro (robot description, xacro)
@@ -30,4 +30,8 @@
   <xacro:frame name="lidar3d_row" parent_link="default_mount">
     <origin xyz="0.0 -1.5 0.0" rpy="0.0 0.0 0.0"/>
+  </xacro:frame>
+  <xacro:include filename="$(find clearpath_platform_description)/urdf/links/frame.urdf.xacro"/>
+  <xacro:frame name="ptu_row" parent_link="default_mount">
+    <origin xyz="0.0 -1.75 0.0" rpy="0.0 0.0 0.0"/>
   </xacro:frame>
   <!-- Mounts -->
@@ -218,4 +222,14 @@
     <origin xyz="0.0 0.0 0.25" rpy="0.0 0.0 0.0"/>
   </xacro:fixposition>
+  <!-- ptu_0 -->
+  <xacro:include filename="$(find clearpath_sensors_description)/urdf/flir_ptu.urdf.xacro"/>
+  <xacro:flir_ptu name="ptu_0" parent_link="ptu_row_link" model="ptu5">
+    <origin xyz="0.0 0.0 0.0" rpy="0.0 0.0 0.0"/>
+  </xacro:flir_ptu>
+  <!-- ptu_1 -->
+  <xacro:include filename="$(find clearpath_sensors_description)/urdf/flir_ptu.urdf.xacro"/>
+  <xacro:flir_ptu name="ptu_1" parent_link="ptu_row_link" model="d46">
+    <origin xyz="0.0 0.0 0.25" rpy="0.0 0.0 0.0"/>
+  </xacro:flir_ptu>
   <!-- Manipulators -->
   <!-- Extras -->
