Commit message: Added samples for UR7e, UR8 Long and UR12e.

File: clearpath_generator_common_tests/samples/test_all_dual_manipulators/robot.srdf.xacro (robot description, xacro)
@@ -71,4 +71,31 @@
   <xacro:include filename="$(find clearpath_manipulators_description)/srdf/arm/universal_robots.srdf.xacro"/>
   <xacro:universal_robots name="arm_22"/>
+  <!-- arm_23 -->
+  <xacro:include filename="$(find clearpath_manipulators_description)/srdf/arm/universal_robots.srdf.xacro"/>
+  <xacro:universal_robots name="arm_23"/>
+  <!-- arm_24 -->
+  <xacro:include filename="$(find clearpath_manipulators_description)/srdf/arm/universal_robots.srdf.xacro"/>
+  <xacro:universal_robots name="arm_24"/>
+  <!-- arm_25 -->
+  <xacro:include filename="$(find clearpath_manipulators_description)/srdf/arm/universal_robots.srdf.xacro"/>
+  <xacro:universal_robots name="arm_25"/>
+  <!-- arm_26 -->
+  <xacro:include filename="$(find clearpath_manipulators_description)/srdf/arm/universal_robots.srdf.xacro"/>
+  <xacro:universal_robots name="arm_26"/>
+  <!-- arm_27 -->
+  <xacro:include filename="$(find clearpath_manipulators_description)/srdf/arm/universal_robots.srdf.xacro"/>
+  <xacro:universal_robots name="arm_27"/>
+  <!-- arm_28 -->
+  <xacro:include filename="$(find clearpath_manipulators_description)/srdf/arm/universal_robots.srdf.xacro"/>
+  <xacro:universal_robots name="arm_28"/>
+  <!-- arm_29 -->
+  <xacro:include filename="$(find clearpath_manipulators_description)/srdf/arm/universal_robots.srdf.xacro"/>
+  <xacro:universal_robots name="arm_29"/>
+  <!-- arm_30 -->
+  <xacro:include filename="$(find clearpath_manipulators_description)/srdf/arm/universal_robots.srdf.xacro"/>
+  <xacro:universal_robots name="arm_30"/>
+  <!-- arm_31 -->
+  <xacro:include filename="$(find clearpath_manipulators_description)/srdf/arm/universal_robots.srdf.xacro"/>
+  <xacro:universal_robots name="arm_31"/>
   <!-- Grippers -->
   <!-- arm_0_gripper -->
@@ -123,4 +150,22 @@
   <xacro:include filename="$(find clearpath_manipulators_description)/srdf/gripper/robotiq_2f_140.srdf.xacro"/>
   <xacro:robotiq_2f_140 name="arm_22_gripper" padding="true"/>
+  <!-- arm_24_gripper -->
+  <xacro:include filename="$(find clearpath_manipulators_description)/srdf/gripper/robotiq_2f_85.srdf.xacro"/>
+  <xacro:robotiq_2f_85 name="arm_24_gripper"/>
+  <!-- arm_25_gripper -->
+  <xacro:include filename="$(find clearpath_manipulators_description)/srdf/gripper/robotiq_2f_140.srdf.xacro"/>
+  <xacro:robotiq_2f_140 name="arm_25_gripper" padding="true"/>
+  <!-- arm_27_gripper -->
+  <xacro:include filename="$(find clearpath_manipulators_description)/srdf/gripper/robotiq_2f_85.srdf.xacro"/>
+  <xacro:robotiq_2f_85 name="arm_27_gripper"/>
+  <!-- arm_28_gripper -->
+  <xacro:include filename="$(find clearpath_manipulators_description)/srdf/gripper/robotiq_2f_140.srdf.xacro"/>
+  <xacro:robotiq_2f_140 name="arm_28_gripper" padding="true"/>
+  <!-- arm_30_gripper -->
+  <xacro:include filename="$(find clearpath_manipulators_description)/srdf/gripper/robotiq_2f_85.srdf.xacro"/>
+  <xacro:robotiq_2f_85 name="arm_30_gripper"/>
+  <!-- arm_31_gripper -->
+  <xacro:include filename="$(find clearpath_manipulators_description)/srdf/gripper/robotiq_2f_140.srdf.xacro"/>
+  <xacro:robotiq_2f_140 name="arm_31_gripper" padding="true"/>
   <!-- Lifts -->
   <!-- lift_0 -->

File: clearpath_generator_common_tests/samples/test_all_dual_manipulators/robot.urdf.xacro (robot description, xacro)
@@ -42,4 +42,8 @@
   <xacro:frame name="ur_row_2" parent_link="default_mount">
     <origin xyz="0.0 -2.0 0.0" rpy="0.0 0.0 0.0"/>
+  </xacro:frame>
+  <xacro:include filename="$(find clearpath_platform_description)/urdf/links/frame.urdf.xacro"/>
+  <xacro:frame name="ur_row_3" parent_link="default_mount">
+    <origin xyz="0.0 -4.0 0.0" rpy="0.0 0.0 0.0"/>
   </xacro:frame>
   <!-- Mounts -->
@@ -161,4 +165,49 @@
     <origin xyz="5.0 0.0 0.0" rpy="0.0 0.0 -1.5707"/>
   </xacro:universal_robots>
+  <!-- arm_23 -->
+  <xacro:include filename="$(find clearpath_manipulators_description)/urdf/arm/universal_robots.urdf.xacro"/>
+  <xacro:universal_robots name="arm_23" parent_link="ur_row_3_link" ur_type="ur7e" robot_ip="192.168.131.40">
+    <origin xyz="0.0 0.0 0.0" rpy="0.0 0.0 -1.5707"/>
+  </xacro:universal_robots>
+  <!-- arm_24 -->
+  <xacro:include filename="$(find clearpath_manipulators_description)/urdf/arm/universal_robots.urdf.xacro"/>
+  <xacro:universal_robots name="arm_24" parent_link="ur_row_3_link" ur_type="ur7e" robot_ip="192.168.131.40">
+    <origin xyz="0.5 0.0 0.0" rpy="0.0 0.0 -1.5707"/>
+  </xacro:universal_robots>
+  <!-- arm_25 -->
+  <xacro:include filename="$(find clearpath_manipulators_description)/urdf/arm/universal_robots.urdf.xacro"/>
+  <xacro:universal_robots name="arm_25" parent_link="ur_row_3_link" ur_type="ur7e" robot_ip="192.168.131.40">
+    <origin xyz="1.0 0.0 0.0" rpy="0.0 0.0 -1.5707"/>
+  </xacro:universal_robots>
+  <!-- arm_26 -->
+  <xacro:include filename="$(find clearpath_manipulators_description)/urdf/arm/universal_robots.urdf.xacro"/>
+  <xacro:universal_robots name="arm_26" parent_link="ur_row_3_link" ur_type="ur8long" robot_ip="192.168.131.40">
+    <origin xyz="2.0 0.0 0.0" rpy="0.0 0.0 -1.5707"/>
+  </xacro:universal_robots>
+  <!-- arm_27 -->
+  <xacro:include filename="$(find clearpath_manipulators_description)/urdf/arm/universal_robots.urdf.xacro"/>
+  <xacro:universal_robots name="arm_27" parent_link="ur_row_3_link" ur_type="ur8long" robot_ip="192.168.131.40">
+    <origin xyz="2.5 0.0 0.0" rpy="0.0 0.0 -1.5707"/>
+  </xacro:universal_robots>
+  <!-- arm_28 -->
+  <xacro:include filename="$(find clearpath_manipulators_description)/urdf/arm/universal_robots.urdf.xacro"/>
+  <xacro:universal_robots name="arm_28" parent_link="ur_row_3_link" ur_type="ur8long" robot_ip="192.168.131.40">
+    <origin xyz="3.0 0.0 0.0" rpy="0.0 0.0 -1.5707"/>
+  </xacro:universal_robots>
+  <!-- arm_29 -->
+  <xacro:include filename="$(find clearpath_manipulators_description)/urdf/arm/universal_robots.urdf.xacro"/>
+  <xacro:universal_robots name="arm_29" parent_link="ur_row_3_link" ur_type="ur12e" robot_ip="192.168.131.40">
+    <origin xyz="4.0 0.0 0.0" rpy="0.0 0.0 -1.5707"/>
+  </xacro:universal_robots>
+  <!-- arm_30 -->
+  <xacro:include filename="$(find clearpath_manipulators_description)/urdf/arm/universal_robots.urdf.xacro"/>
+  <xacro:universal_robots name="arm_30" parent_link="ur_row_3_link" ur_type="ur12e" robot_ip="192.168.131.40">
+    <origin xyz="4.5 0.0 0.0" rpy="0.0 0.0 -1.5707"/>
+  </xacro:universal_robots>
+  <!-- arm_31 -->
+  <xacro:include filename="$(find clearpath_manipulators_description)/urdf/arm/universal_robots.urdf.xacro"/>
+  <xacro:universal_robots name="arm_31" parent_link="ur_row_3_link" ur_type="ur12e" robot_ip="192.168.131.40">
+    <origin xyz="5.0 0.0 0.0" rpy="0.0 0.0 -1.5707"/>
+  </xacro:universal_robots>
   <!-- lift_0 -->
   <xacro:include filename="$(find clearpath_manipulators_description)/urdf/lift/ewellix.urdf.xacro"/>
@@ -301,4 +350,34 @@
     <origin xyz="0.0 0.0 0.0" rpy="0.0 0.0 0.0"/>
   </xacro:robotiq_2f_140>
+  <!-- arm_24_gripper -->
+  <xacro:include filename="$(find clearpath_manipulators_description)/urdf/gripper/robotiq_2f_85.urdf.xacro"/>
+  <xacro:robotiq_2f_85 name="arm_24_gripper" parent_link="arm_24_tool0">
+    <origin xyz="0.0 0.0 0.0" rpy="0.0 0.0 0.0"/>
+  </xacro:robotiq_2f_85>
+  <!-- arm_25_gripper -->
+  <xacro:include filename="$(find clearpath_manipulators_description)/urdf/gripper/robotiq_2f_140.urdf.xacro"/>
+  <xacro:robotiq_2f_140 name="arm_25_gripper" parent_link="arm_25_tool0">
+    <origin xyz="0.0 0.0 0.0" rpy="0.0 0.0 0.0"/>
+  </xacro:robotiq_2f_140>
+  <!-- arm_27_gripper -->
+  <xacro:include filename="$(find clearpath_manipulators_description)/urdf/gripper/robotiq_2f_85.urdf.xacro"/>
+  <xacro:robotiq_2f_85 name="arm_27_gripper" parent_link="arm_27_tool0">
+    <origin xyz="0.0 0.0 0.0" rpy="0.0 0.0 0.0"/>
+  </xacro:robotiq_2f_85>
+  <!-- arm_28_gripper -->
+  <xacro:include filename="$(find clearpath_manipulators_description)/urdf/gripper/robotiq_2f_140.urdf.xacro"/>
+  <xacro:robotiq_2f_140 name="arm_28_gripper" parent_link="arm_28_tool0">
+    <origin xyz="0.0 0.0 0.0" rpy="0.0 0.0 0.0"/>
+  </xacro:robotiq_2f_140>
+  <!-- arm_30_gripper -->
+  <xacro:include filename="$(find clearpath_manipulators_description)/urdf/gripper/robotiq_2f_85.urdf.xacro"/>
+  <xacro:robotiq_2f_85 name="arm_30_gripper" parent_link="arm_30_tool0">
+    <origin xyz="0.0 0.0 0.0" rpy="0.0 0.0 0.0"/>
+  </xacro:robotiq_2f_85>
+  <!-- arm_31_gripper -->
+  <xacro:include filename="$(find clearpath_manipulators_description)/urdf/gripper/robotiq_2f_140.urdf.xacro"/>
+  <xacro:robotiq_2f_140 name="arm_31_gripper" parent_link="arm_31_tool0">
+    <origin xyz="0.0 0.0 0.0" rpy="0.0 0.0 0.0"/>
+  </xacro:robotiq_2f_140>
   <!-- Extras -->
 </robot>
